File: hub.sch (KiCad schematic (older format))
At the start: 23 parts, among them J1 USB_C_Receptacle_USB2.0, J6 Conn_01x03, U14 GL850G, U15 K24C02D-O, X2 ECS-2520MV-120-xx

Commit message: sch: List LCSC P/N for each component
Parts:
- C34, C35, C36, C37, C38, C39, C40, C42: LCSC P/N (none) -> C1591; MFR P/N (none) -> CL10B104KB8NNNC
- C41: LCSC P/N (none) -> C1644; MFR P/N (none) -> CL10C150JB8NNNC
- FB1: LCSC P/N (none) -> C136491; MFR P/N (none) -> MMZ1608Y601BTA00
- J1: LCSC P/N (none) -> C165948; MFR P/N (none) -> TYPE-C-31-M-12
- J6: LCSC P/N (none) -> C49257; MFR P/N (none) -> C49257
- R19, R34, R35, R36: LCSC P/N (none) -> C115324; MFR P/N (none) -> RS-03K1002FT
- R20: LCSC P/N (none) -> C88607; MFR P/N (none) -> RS-03K6800FT
- R3, R4: LCSC P/N (none) -> C156350; MFR P/N (none) -> RS-03K5101FT
- R33: LCSC P/N (none) -> C327826; MFR P/N (none) -> MR06X1003FTL
- U14: LCSC P/N (none) -> C127278; MFR P/N (none) -> GL850G-OHY37
- U15: LCSC P/N (none) -> C84964; MFR P/N (none) -> K24C02
- X2: LCSC P/N (none) -> C405460; MFR P/N (none) -> ECS-2520MV-120-BN-TR
Changed lines of the file:
@@
 F 2 "Package_DFN_QFN:QFN-28-1EP_5x5mm_P0.5mm_EP3.35x3.35mm_ThermalVias" H 6450 3700 50  0001 C CNN
 F 3 "https://www.kean.com.au/oshw/WR703N/GL850G%20USB%20Hub%201.07.pdf" H 6450 3200 50  0001 C CNN
+F 4 "C127278" H 6450 3200 50  0001 C CNN "LCSC P/N"
+F 5 "GL850G-OHY37" H 6450 3200 50  0001 C CNN "MFR P/N"
 	1    6450 3200
 	1    0    0    -1
@@
 F 2 "Oscillator:Oscillator_SMD_ECS_2520MV-xxx-xx-4Pin_2.5x2.0mm" H 3850 4850 50  0001 C CNN
 F 3 "https://www.ecsxtal.com/store/pdf/ECS-2520MV.pdf" H 3225 5325 50  0001 C CNN
+F 4 "C405460" H 3400 5200 50  0001 C CNN "LCSC P/N"
+F 5 "ECS-2520MV-120-BN-TR" H 3400 5200 50  0001 C CNN "MFR P/N"
 	1    3400 5200
 	1    0    0    -1
@@
 F 2 "antboard:USB_C_Receptacle_Palconn_UTC16-G" H 3600 3300 50  0001 C CNN
 F 3 "https://www.usb.org/sites/default/files/documents/usb_type-c.zip" H 3600 3300 50  0001 C CNN
+F 4 "C165948" H 3450 3300 50  0001 C CNN "LCSC P/N"
+F 5 "TYPE-C-31-M-12" H 3450 3300 50  0001 C CNN "MFR P/N"
 	1    3450 3300
 	1    0    0    -1
@@
 F 2 "Resistor_SMD:R_0603_1608Metric" H 4250 2900 50  0001 C CNN
 F 3 "~" H 4250 2900 50  0001 C CNN
+F 4 "C156350" H 4250 2900 50  0001 C CNN "LCSC P/N"
+F 5 "RS-03K5101FT" H 4250 2900 50  0001 C CNN "MFR P/N"
 	1    4250 2900
 	0    1    1    0
@@
 F 2 "Resistor_SMD:R_0603_1608Metric" H 4250 3000 50  0001 C CNN
 F 3 "~" H 4250 3000 50  0001 C CNN
+F 4 "C156350" H 4250 3000 50  0001 C CNN "LCSC P/N"
+F 5 "RS-03K5101FT" H 4250 3000 50  0001 C CNN "MFR P/N"
 	1    4250 3000
 	0    1    -1   0
@@
 F 2 "Resistor_SMD:R_0603_1608Metric" H 6150 4400 50  0001 C CNN
 F 3 "~" H 6150 4400 50  0001 C CNN
+F 4 "C88607" H 6150 4400 50  0001 C CNN "LCSC P/N"
+F 5 "RS-03K6800FT" H 6150 4400 50  0001 C CNN "MFR P/N"
 	1    6150 4400
 	0    1    1    0
@@
 F 2 "Capacitor_SMD:C_0603_1608Metric" H 5950 4150 50  0001 C CNN
 F 3 "~" H 5950 4150 50  0001 C CNN
+F 4 "C1591" H 5950 4150 50  0001 C CNN "LCSC P/N"
+F 5 "CL10B104KB8NNNC" H 5950 4150 50  0001 C CNN "MFR P/N"
 	1    5950 4150
 	1    0    0    1
@@
 F 2 "Resistor_SMD:R_0603_1608Metric" H 5750 3900 50  0001 C CNN
 F 3 "~" H 5750 3900 50  0001 C CNN
+F 4 "C115324" H 5750 3900 50  0001 C CNN "LCSC P/N"
+F 5 "RS-03K1002FT" H 5750 3900 50  0001 C CNN "MFR P/N"
 	1    5750 3900
 	0    -1   -1   0
@@
 F 2 "Resistor_SMD:R_0603_1608Metric" H 2900 5000 50  0001 C CNN
 F 3 "~" H 2900 5000 50  0001 C CNN
+F 4 "C327826" H 2900 5000 50  0001 C CNN "LCSC P/N"
+F 5 "MR06X1003FTL" H 2900 5000 50  0001 C CNN "MFR P/N"
 	1    2900 5000
 	1    0    0    -1
@@
 F 2 "Capacitor_SMD:C_0603_1608Metric" H 3900 5400 50  0001 C CNN
 F 3 "~" H 3900 5400 50  0001 C CNN
+F 4 "C1644" H 3900 5400 50  0001 C CNN "LCSC P/N"
+F 5 "CL10C150JB8NNNC" H 3900 5400 50  0001 C CNN "MFR P/N"
 	1    3900 5400
 	1    0    0    1
@@
 F 2 "Inductor_SMD:L_0603_1608Metric" V 6080 1800 50  0001 C CNN
 F 3 "~" H 6150 1800 50  0001 C CNN
+F 4 "C136491" H 6150 1800 50  0001 C CNN "LCSC P/N"
+F 5 "MMZ1608Y601BTA00" H 6150 1800 50  0001 C CNN "MFR P/N"
 	1    6150 1800
 	0    -1   -1   0
@@
 F 2 "Capacitor_SMD:C_0603_1608Metric" H 5850 2000 50  0001 C CNN
 F 3 "~" H 5850 2000 50  0001 C CNN
+F 4 "C1591" H 5850 2000 50  0001 C CNN "LCSC P/N"
+F 5 "CL10B104KB8NNNC" H 5850 2000 50  0001 C CNN "MFR P/N"
 	1    5850 2000
 	1    0    0    1
@@
 F 2 "Capacitor_SMD:C_0603_1608Metric" H 6500 2000 50  0001 C CNN
 F 3 "~" H 6500 2000 50  0001 C CNN
+F 4 "C1591" H 6500 2000 50  0001 C CNN "LCSC P/N"
+F 5 "CL10B104KB8NNNC" H 6500 2000 50  0001 C CNN "MFR P/N"
 	1    6500 2000
 	1    0    0    1
@@
 F 2 "Capacitor_SMD:C_0603_1608Metric" H 6900 2000 50  0001 C CNN
 F 3 "~" H 6900 2000 50  0001 C CNN
+F 4 "C1591" H 6900 2000 50  0001 C CNN "LCSC P/N"
+F 5 "CL10B104KB8NNNC" H 6900 2000 50  0001 C CNN "MFR P/N"
 	1    6900 2000
 	1    0    0    1
@@
 F 2 "Capacitor_SMD:C_0603_1608Metric" H 7300 2000 50  0001 C CNN
 F 3 "~" H 7300 2000 50  0001 C CNN
+F 4 "C1591" H 7300 2000 50  0001 C CNN "LCSC P/N"
+F 5 "CL10B104KB8NNNC" H 7300 2000 50  0001 C CNN "MFR P/N"
 	1    7300 2000
 	1    0    0    1
@@
 F 2 "Capacitor_SMD:C_0603_1608Metric" H 7700 2000 50  0001 C CNN
 F 3 "~" H 7700 2000 50  0001 C CNN
+F 4 "C1591" H 7700 2000 50  0001 C CNN "LCSC P/N"
+F 5 "CL10B104KB8NNNC" H 7700 2000 50  0001 C CNN "MFR P/N"
 	1    7700 2000
 	1    0    0    1
@@
 F 2 "Capacitor_SMD:C_0603_1608Metric" H 8100 2000 50  0001 C CNN
 F 3 "~" H 8100 2000 50  0001 C CNN
+F 4 "C1591" H 8100 2000 50  0001 C CNN "LCSC P/N"
+F 5 "CL10B104KB8NNNC" H 8100 2000 50  0001 C CNN "MFR P/N"
 	1    8100 2000
 	1    0    0    1
@@
 F 2 "Capacitor_SMD:C_0603_1608Metric" H 8500 2000 50  0001 C CNN
 F 3 "~" H 8500 2000 50  0001 C CNN
+F 4 "C1591" H 8500 2000 50  0001 C CNN "LCSC P/N"
+F 5 "CL10B104KB8NNNC" H 8500 2000 50  0001 C CNN "MFR P/N"
 	1    8500 2000
 	1    0    0    1
@@
 F 2 "Package_TO_SOT_SMD:SOT-23-5" H 5800 5850 50  0001 C CNN
 F 3 "https://datasheet.lcsc.com/szlcsc/1809261012_Hua-Hong-NEC-K24C02_C84964.pdf" H 5800 5850 50  0001 C CNN
+F 4 "C84964" H 5800 5850 50  0001 C CNN "LCSC P/N"
+F 5 "K24C02" H 5800 5850 50  0001 C CNN "MFR P/N"
 	1    5800 5850
 	1    0    0    -1
@@
 F 2 "Resistor_SMD:R_0603_1608Metric" H 5400 5750 50  0001 C CNN
 F 3 "~" H 5400 5750 50  0001 C CNN
+F 4 "C115324" H 5400 5750 50  0001 C CNN "LCSC P/N"
+F 5 "RS-03K1002FT" H 5400 5750 50  0001 C CNN "MFR P/N"
 	1    5400 5750
 	1    0    0    -1
@@
 F 2 "Connector_PinHeader_2.54mm:PinHeader_1x03_P2.54mm_Vertical" H 4500 6050 50  0001 C CNN
 F 3 "~" H 4500 6050 50  0001 C CNN
+F 4 "C49257" H 4500 6050 50  0001 C CNN "LCSC P/N"
+F 5 "C49257" H 4500 6050 50  0001 C CNN "MFR P/N"
 	1    4500 6050
 	-1   0    0    -1
@@
 F 2 "Resistor_SMD:R_0603_1608Metric" H 5500 5750 50  0001 C CNN
 F 3 "~" H 5500 5750 50  0001 C CNN
+F 4 "C115324" H 5500 5750 50  0001 C CNN "LCSC P/N"
+F 5 "RS-03K1002FT" H 5500 5750 50  0001 C CNN "MFR P/N"
 	1    5500 5750
 	1    0    0    -1
@@
 F 2 "Resistor_SMD:R_0603_1608Metric" H 5750 4600 50  0001 C CNN
 F 3 "~" H 5750 4600 50  0001 C CNN
+F 4 "C115324" H 5750 4600 50  0001 C CNN "LCSC P/N"
+F 5 "RS-03K1002FT" H 5750 4600 50  0001 C CNN "MFR P/N"
 	1    5750 4600
 	0    -1   -1   0
