File: io.sch (KiCad schematic (older format))
At the start: 7 parts, among them J3 Conn_02x05_Odd_Even, J4 Conn_02x10_Odd_Even, J5 Conn_02x05_Odd_Even, U10 TXB0104PW, U7 TXB0108DQSR, U8 TXB0108DQSR, U9 TXB0108DQSR

Commit message: sch: List LCSC P/N for each component
Parts:
- J3, J5: LCSC P/N (none) -> C150517; MFR P/N (none) -> 20021121-00010C4LF
- J4: LCSC P/N (none) -> C59981; MFR P/N (none) -> C59981
- U10: LCSC P/N (none) -> C60708; MFR P/N (none) -> TXB0104PWR
- U7, U8, U9: LCSC P/N (none) -> C53406; MFR P/N (none) -> TXB0108PWR
Changed lines of the file:
@@
 F 2 "Package_SO:TSSOP-14_4.4x5mm_P0.65mm" H 3800 4100 50  0001 C CNN
 F 3 "http://www.ti.com/lit/ds/symlink/txb0104.pdf" H 3910 4945 50  0001 C CNN
+F 4 "C60708" H 3800 4850 50  0001 C CNN "LCSC P/N"
+F 5 "TXB0104PWR" H 3800 4850 50  0001 C CNN "MFR P/N"
 	1    3800 4850
 	1    0    0    -1
@@
 F 2 "Package_SO:TSSOP-20_4.4x6.5mm_P0.65mm" H 3800 2050 50  0001 C CNN
 F 3 "http://www.ti.com/lit/ds/symlink/txb0108.pdf" H 3800 2700 50  0001 C CNN
+F 4 "C53406" H 3800 2800 50  0001 C CNN "LCSC P/N"
+F 5 "TXB0108PWR" H 3800 2800 50  0001 C CNN "MFR P/N"
 	1    3800 2800
 	1    0    0    -1
@@
 F 2 "Connector_PinHeader_1.27mm:PinHeader_2x05_P1.27mm_Vertical_SMD" H 9300 4700 50  0001 C CNN
 F 3 "~" H 9300 4700 50  0001 C CNN
+F 4 "C150517" H 9300 4700 50  0001 C CNN "LCSC P/N"
+F 5 "20021121-00010C4LF" H 9300 4700 50  0001 C CNN "MFR P/N"
 	1    9300 4700
 	1    0    0    -1
@@
 F 2 "Package_SO:TSSOP-20_4.4x6.5mm_P0.65mm" H 8500 4050 50  0001 C CNN
 F 3 "http://www.ti.com/lit/ds/symlink/txb0108.pdf" H 8500 4700 50  0001 C CNN
+F 4 "C53406" H 8500 4800 50  0001 C CNN "LCSC P/N"
+F 5 "TXB0108PWR" H 8500 4800 50  0001 C CNN "MFR P/N"
 	1    8500 4800
 	1    0    0    -1
@@
 F 2 "Connector_PinHeader_1.27mm:PinHeader_2x05_P1.27mm_Vertical_SMD" H 9300 2550 50  0001 C CNN
 F 3 "~" H 9300 2550 50  0001 C CNN
+F 4 "C150517" H 9300 2550 50  0001 C CNN "LCSC P/N"
+F 5 "20021121-00010C4LF" H 9300 2550 50  0001 C CNN "MFR P/N"
 	1    9300 2550
 	1    0    0    -1
@@
 F 2 "Package_SO:TSSOP-20_4.4x6.5mm_P0.65mm" H 8500 1900 50  0001 C CNN
 F 3 "http://www.ti.com/lit/ds/symlink/txb0108.pdf" H 8500 2550 50  0001 C CNN
+F 4 "C53406" H 8500 2650 50  0001 C CNN "LCSC P/N"
+F 5 "TXB0108PWR" H 8500 2650 50  0001 C CNN "MFR P/N"
 	1    8500 2650
 	1    0    0    -1
@@
 F 2 "Connector_PinHeader_1.27mm:PinHeader_2x10_P1.27mm_Vertical_SMD" H 5300 3800 50  0001 C CNN
 F 3 "~" H 5300 3800 50  0001 C CNN
+F 4 "C59981" H 5300 3800 50  0001 C CNN "LCSC P/N"
+F 5 "C59981" H 5300 3800 50  0001 C CNN "MFR P/N"
 	1    5300 3800
 	1    0    0    -1
